File: flex/flex.kicad_pcb (KiCad board)
At the start: 2 copper layers, 126.3 x 113 mm, 105 parts, among them J1 Conn_01x06_Female, J2 Conn_01x05_Female, J3 Conn_01x03_Female, J4 Conn_01x06_Female, J5 Conn_01x03_Female, SW1 SW_Push, SW10 SW_Push, SW11 SW_Push, SW12 SW_Push, SW14 SW_Push, SW15 SW_Push, SW16 SW_Push, SW17 SW_Push, SW19 SW_Push, SW2 SW_Push, SW20 SW_Push, SW21 SW_Push, SW22 SW_Push, SW23 SW_Push, SW24 SW_Push, SW25 SW_Push, SW26 SW_Push, SW3 SW_Push, SW4 SW_Push, SW5 SW_Push, SW6 SW_Push, SW7 SW_Push, SW8 SW_Push, SW9 SW_Push

Commit message: edge cuts, via size
Parts:
- moved D10 11.2 mm to (92.4, 78.3)
Routing:
- net col1: track 286.2 -> 288.9 mm
- net col2: track 273.9 -> 276.4 mm
- net row4: track 431.6 -> 433.8 mm
- net Vcc: track 930.8 -> 933.0 mm
- net Net-(D37-Pad1): track 38.3 -> 40.1 mm
- net col4: track 132.9 -> 134.7 mm
- net Net-(D10-Pad2): track 14.1 -> 15.1 mm
- net row5: track 45.7 -> 46.7 mm
- net Net-(D25-Pad1): track 125.9 -> 125.0 mm
- net row3: track 263.9 -> 264.7 mm
- net Net-(D23-Pad1): track 38.2 -> 38.9 mm
- net Net-(D5-Pad1): track 40.3 -> 39.8 mm
Other:
- outline, holes or cut-outs redrawn

Commit message: cleanup
Parts:
- moved D10 11.2 mm to (81.4, 80.4)
Routing:
- net col5: track 160.8 -> 134.3 mm, vias 3 -> 2
- net Vcc: track 933.0 -> 946.2 mm
- net row1: track 658.5 -> 667.4 mm
- net row3: track 264.7 -> 271.6 mm
- net row2: track 502.8 -> 509.6 mm
- net Net-(D19-Pad3): track 164.0 -> 170.7 mm
- net row4: track 433.8 -> 439.6 mm
- net Net-(D18-Pad1): track 122.4 -> 127.3 mm
- net Net-(D55-Pad1): track 42.8 -> 45.6 mm
- net Gnd: track 898.7 -> 901.1 mm
- net Net-(D10-Pad2): track 15.1 -> 13.0 mm
- net Net-(D53-Pad1): track 38.9 -> 40.9 mm
- net Net-(D2-Pad1): track 37.7 -> 39.7 mm
- net Net-(D49-Pad1): track 39.7 -> 41.5 mm
- net col1: track 288.9 -> 290.6 mm
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Other:
- outline, holes or cut-outs redrawn

Commit message: revert routing
Routing:
- net col5: track 134.3 -> 160.8 mm, vias 2 -> 3
- net Vcc: track 946.2 -> 930.8 mm
- net row1: track 667.4 -> 658.5 mm
- net row4: track 439.6 -> 431.6 mm
- net row3: track 271.6 -> 263.9 mm
- net row2: track 509.6 -> 502.7 mm
- net Net-(D19-Pad3): track 170.7 -> 164.0 mm
- net Net-(D18-Pad1): track 127.3 -> 122.4 mm
- net col1: track 290.6 -> 286.2 mm
- net Gnd: track 901.1 -> 898.2 mm
- net Net-(D55-Pad1): track 45.6 -> 42.8 mm
- net col2: track 276.1 -> 273.9 mm
- net Net-(D53-Pad1): track 40.9 -> 38.9 mm
- net Net-(D2-Pad1): track 39.7 -> 37.7 mm
- net col4: track 134.8 -> 132.9 mm
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Other:
- board text added: "Conn_01x06_Female"
- board text added: "Conn_01x07_Female"
- board text added: "D"
- board text added: "J1"
- board text added: "J10"
- board text added: "J11"
- board text added: "J12"
- board text added: "J13"
- board text added: "J14"
- board text added: "J15"
- board text added: "J2"
- board text added: "J3"
- board text added: "J4"
- board text added: "J5"
- board text added: "J6"
- board text added: "J7"
- board text added: "J8"
- board text added: "J9"
- board text added: "REV 2.46"
- board text added: "SW1"
- board text added: "SW10"
- board text added: "SW11"
- board text added: "SW12"
- board text added: "SW13"
- board text added: "SW14"
- board text added: "SW15"
- board text added: "SW16"
- board text added: "SW17"
- board text added: "SW18"
- board text added: "SW19"
- board text added: "SW2"
- board text added: "SW20"
- board text added: "SW21"
- board text added: "SW22"
- board text added: "SW23"
- board text added: "SW24"
- board text added: "SW25"
- board text added: "SW26"
- board text added: "SW27"
- board text added: "SW28"
- board text added: "SW29"
- board text added: "SW3"
- board text added: "SW30"
- board text added: "SW31"
- board text added: "SW32"
- board text added: "SW4"
- board text added: "SW5"
- board text added: "SW6"
- board text added: "SW7"
- board text added: "SW8"
- board text added: "SW9"
- board text added: "SW_Push"
- board text removed: "REV 2.5"

Commit message: silkscreen
Other:
- board text added: "REV 2.47"
- board text removed: "REV 2.46"
Changed lines of the file:
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@@
   (gr_arc (start 150.133 122.941987) (mid 150.385093 122.970144) (end 150.62447 123.054065) (layer "Edge.Cuts") (width 0.2))
   (gr_line (start 94.725201 81.359399) (end 94.736482 119.144) (layer "Edge.Cuts") (width 0.2))
-  (gr_arc (start 127.709702 34.842393) (mid 126.7752 34.4644) (end 126.369517 33.541582) (layer "Edge.Cuts") (width 0.2))
+  (gr_arc (start 127.709702 34.842393) (mid 126.775201 34.4644) (end 126.369517 33.541582) (layer "Edge.Cuts") (width 0.2))
   (gr_circle (center 107.567997 33.58029) (end 107.967997 33.58029) (layer "Edge.Cuts") (width 0.2) (fill none))
   (gr_line (start 86.713285 102.809399) (end 78.4252 102.8094) (layer "Edge.Cuts") (width 0.2))
@@
   (gr_arc (start 156.88153 36.951921) (mid 156.252977 37.381695) (end 156.512309 36.665782) (layer "Edge.Cuts") (width 0.2))
   (gr_arc (start 35.9252 133.184399) (mid 35.571647 133.037952) (end 35.4252 132.684399) (layer "Edge.Cuts") (width 0.2))
-  (gr_arc (start 70.326156 35.604585) (mid 70.926966 34.1644) (end 72.3752 33.583262) (layer "Edge.Cuts") (width 0.2))
+  (gr_arc (start 70.326156 35.604585) (mid 70.926966 34.164401) (end 72.3752 33.583262) (layer "Edge.Cuts") (width 0.2))
   (gr_arc (start 83.619083 33.595785) (mid 84.640406 34.244827) (end 84.482308 35.444561) (layer "Edge.Cuts") (width 0.2))
   (gr_line (start 110.811975 123.365623) (end 110.813692 119.811424) (layer "Edge.Cuts") (width 0.05))
@@
   (gr_line (start 150.619083 34.825785) (end 136.07407 34.840294) (layer "Edge.Cuts") (width 0.2))
   (gr_line (start 145.9352 104.054401) (end 145.9352 109.9044) (layer "Edge.Cuts") (width 0.05))
-  (gr_arc (start 125.040698 31.286407) (mid 125.9752 31.6644) (end 126.380883 32.587218) (layer "Edge.Cuts") (width 0.2))
+  (gr_arc (start 125.040698 31.286407) (mid 125.975199 31.6644) (end 126.380883 32.587218) (layer "Edge.Cuts") (width 0.2))
   (gr_line (start 118.4752 101.0594) (end 118.4752 103.559399) (layer "Edge.Cuts") (width 0.2))
   (gr_line (start 44.2252 86.6594) (end 50.725201 86.6594) (layer "Edge.Cuts") (width 0.2))
@@
   (gr_line (start 116.7414 119.910798) (end 116.7346 120.9896) (layer "Edge.Cuts") (width 0.05))
   (gr_line (start 78.9252 119.143999) (end 78.9252 104.3094) (layer "Edge.Cuts") (width 0.2))
-  (gr_arc (start 92.274389 32.704585) (mid 92.652382 31.770083) (end 93.5752 31.3644) (layer "Edge.Cuts") (width 0.2))
+  (gr_arc (start 92.274389 32.704585) (mid 92.652382 31.770084) (end 93.5752 31.3644) (layer "Edge.Cuts") (width 0.2))
   (gr_line (start 65.7252 109.609398) (end 72.2252 109.609399) (layer "Edge.Cuts") (width 0.2))
   (gr_line (start 132.2252 98.859399) (end 124.925199 98.859399) (layer "Edge.Cuts") (width 0.2))
@@
   (gr_arc (start 65.725201 115.809398) (mid 65.225201 115.309398) (end 65.725201 114.809398) (layer "Edge.Cuts") (width 0.2))
   (gr_circle (center 132.123002 122.94618) (end 131.723002 122.94618) (layer "Edge.Cuts") (width 0.2) (fill none))
-  (gr_arc (start 81.736115 125.245961) (mid 82.114108 124.311459) (end 83.036926 123.905776) (layer "Edge.Cuts") (width 0.2))
+  (gr_arc (start 81.736115 125.245961) (mid 82.114108 124.31146) (end 83.036926 123.905776) (layer "Edge.Cuts") (width 0.2))
   (gr_arc (start 111.181912 119.523999) (mid 111.420994 119.439243) (end 111.672988 119.410206) (layer "Edge.Cuts") (width 0.2))
   (gr_arc (start 84.114088 35.731987) (mid 83.875006 35.816743) (end 83.623012 35.84578) (layer "Edge.Cuts") (width 0.2))
@@
     (effects (font (size 1 1) (thickness 0.15)) (justify mirror))
   )
-  (gr_text "REV 2.46" (at 80.9652 100.9244) (layer "B.SilkS")
+  (gr_text "REV 2.47" (at 80.9652 100.9244) (layer "B.SilkS")
     (effects (font (size 0.8 0.8) (thickness 0.12)) (justify mirror))
   )
@@
     (effects (font (size 1 1) (thickness 0.15)))
   )
-  (gr_text "REV 2.46" (at 81.1402 100.9744) (layer "F.SilkS")
-    (effects (font (size 0.8 0.8) (thickness 0.12)))
-  )
+  (gr_text "REV 2.47" (at 81.1402 100.9744) (layer "F.SilkS")
+    (effects (font (size 0.8 0.8) (thickness 0.12)))
+  )
