File: flex/flex.kicad_pcb (KiCad board)
At the start: 4 copper layers, 126.3 x 113 mm, 107 parts, among them J1 Conn_01x06_Female, J2 Conn_01x05_Female, J3 Conn_01x06_Female, J4 Conn_01x03_Female, J5 Conn_01x03_Female, SW1 SW_Push, SW10 SW_Push, SW11 SW_Push, SW12 SW_Push, SW13 SW_Push, SW14 SW_Push, SW15 SW_Push, SW16 SW_Push, SW17 SW_Push, SW18 SW_Push, SW19 SW_Push, SW2 SW_Push, SW20 SW_Push, SW21 SW_Push, SW22 SW_Push, SW23 SW_Push, SW24 SW_Push, SW3 SW_Push, SW4 SW_Push, SW5 SW_Push, SW6 SW_Push, SW7 SW_Push, SW8 SW_Push, SW9 SW_Push

Commit message: routing
Parts:
- moved D55 0.40 mm to (60.0, 110.7)
Routing:
- net Vcc: track 0.00 -> 769.7 mm, vias 0 -> 4
- net col6: track 3.10 -> 262.6 mm, vias 0 -> 3
- net row1: track 424.1 -> 627.7 mm
- net col5: track 3.23 -> 194.4 mm, vias 0 -> 1
- net col1: track 154.6 -> 302.0 mm, vias 1 -> 5
- net Net-(D16-DOUT): track 0.00 -> 132.7 mm
- net row4: track 280.0 -> 409.6 mm, vias 4 -> 5
- net row2: track 282.7 -> 408.8 mm
- net col2: track 249.9 -> 355.0 mm, vias 3 -> 4
- net col3: track 165.3 -> 268.1 mm, vias 3 -> 2
- net row3: track 213.7 -> 293.6 mm
- net row5: track 0.00 -> 58.6 mm
- net Net-(D14-DOUT): track 0.00 -> 39.7 mm
- net Net-(D13-DOUT): track 0.00 -> 30.9 mm, vias 0 -> 2
- net Net-(D15-DOUT): track 0.00 -> 28.8 mm
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Other:
- copper layers 4 -> 2

Commit message: routing
Routing:
- net Net-(D18-DOUT): track 0.00 -> 37.0 mm, vias 0 -> 1
- net Net-(D19-DOUT): track 0.00 -> 35.8 mm

Commit message: routing
Routing:
- net Net-(D20-DOUT): track 0.00 -> 168.2 mm
- net Net-(D40-DOUT): track 0.00 -> 168.1 mm, vias 0 -> 2
- net Net-(D24-DOUT): track 0.00 -> 128.7 mm, vias 0 -> 1
- net Net-(D44-DOUT): track 0.00 -> 118.0 mm, vias 0 -> 1
- net Vcc: track 770.1 -> 836.5 mm, vias 4 -> 8
- net Net-(D38-DOUT): track 0.00 -> 41.8 mm, vias 0 -> 2
- net Net-(D22-DOUT): track 0.00 -> 36.2 mm
- net Net-(D23-DOUT): track 0.00 -> 36.0 mm, vias 0 -> 1
- net Net-(D39-DOUT): track 0.00 -> 36.0 mm
- net Net-(D37-DOUT): track 0.00 -> 34.2 mm, vias 0 -> 2
- net Net-(D21-DOUT): track 0.00 -> 33.1 mm
- net Net-(D42-DOUT): track 0.00 -> 32.5 mm, vias 0 -> 1
- net Net-(D45-DOUT): track 0.00 -> 29.4 mm
- net Net-(D43-DOUT): track 0.00 -> 29.1 mm
- net Net-(D46-DOUT): track 0.00 -> 29.0 mm
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